Commit message: Correct collision of URDF

File: urdf/robot.urdf (robot description, URDF)
Before this commit: robot onshape, 15 links, 14 joints
Links:
- link ll_faa: mass 0.19869954999999994705 -> 0.19869955000000011358; geometry collision box size=0.14000000000000001332 0.055000000000000000278 0.0550000000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; visual mesh filename=package://cal_hum_description/meshs/ll_faa.stl
- link ll_ffe: mass 0.099322750000000029069 -> 0.099322750000000056825; geometry visual mesh filename=package://cal_hum_description/meshs/ll_ffe.stl
- link ll_haa: mass 0.79600000000000037392 -> 0.79600000000000059597; geometry visual mesh filename=package://cal_hum_description/meshs/ll_haa.stl
- link ll_hfe: mass 3.5233394799999993019 -> 3.5233394799999966374; geometry visual mesh filename=package://cal_hum_description/meshs/ll_hfe.stl
- link ll_hr: mass 0.73133287000000002376 -> 0.73133287000000013478; geometry visual mesh filename=package://cal_hum_description/meshs/ll_hr.stl
- link ll_kfe: mass 0.24071601000000017456 -> 0.24071601000000006354; geometry visual mesh filename=package://cal_hum_description/meshs/ll_kfe.stl
- link lr_faa: mass 0.19869955000000003031 -> 0.19869955000000000256; geometry collision box size=0.14000000000000001332 0.055000000000000000278 0.0550000000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; visual mesh filename=package://cal_hum_description/meshs/lr_faa.stl
- link lr_ffe: geometry visual mesh filename=package://cal_hum_description/meshs/lr_ffe.stl
- link lr_haa: mass 0.79599999999999981881 -> 0.79599999999999970779; geometry visual mesh filename=package://cal_hum_description/meshs/lr_haa.stl
- link lr_hfe: geometry visual mesh filename=package://cal_hum_description/meshs/lr_hfe.stl
- link lr_hr: mass 0.73133287000000202216 -> 0.73133287000000080091; geometry visual mesh filename=package://cal_hum_description/meshs/lr_hr.stl
- link lr_kfe: mass 0.24100000000000015854 -> 0.24099999999999996425; geometry visual mesh filename=package://cal_hum_description/meshs/lr_kfe.stl
- link torso: mass 2.9270371599999722712 -> 2.927037159999976268; geometry visual mesh filename=package://cal_hum_description/meshs/torso.stl
Joints:
- joint LL_FAA: origin xyz=1.1102230246251565404e-15 0.020000000000026586788 -1.9428902930940239457e-15 rpy=-1.5707963267948912289 -1.5707963267948901187 0 -> xyz=6.6613381477509392425e-16 0.020000000000026579849 -1.9428902930940239457e-15 rpy=-1.5707963267948634734 -1.5707963267948870101 0
- joint LL_FFE: origin xyz=-0.18000000000000215827 1.0633854907737827489e-14 -4.4964032497318839887e-15 rpy=7.3118594512411069293e-16 -3.8857805861880691907e-15 -2.4841240175987530493e-15 -> xyz=-0.18000000000000204725 7.6709472107694409715e-15 -4.5519144009631418157e-15 rpy=-4.142519660632226433e-15 -2.2343238370579094176e-15 5.9396931817444589069e-15
- joint LL_FOOT_frame: origin xyz=1.3877787807814456755e-15 -0.033000000000000473399 0.020976404179762334068 rpy=-1.570796326794896558 -1.570796326794896558 0 -> xyz=1.360023205165816762e-15 -0.033000000000000473399 0.020976404179762330598 rpy=-1.5707963267948936714 -1.570796326794896558 0
- joint LL_HAA: origin xyz=0.015799999999996143518 -1.360023205165816762e-15 -0.064999999999997906674 rpy=1.300043474638154911e-15 -1.5707963267948870101 0 -> xyz=0.015799999999996153927 -1.360023205165816762e-15 -0.064999999999997906674 rpy=1.2864546617328002073e-15 -1.5707963267948952257 0
- joint LL_HFE: origin xyz=-1.7763568394002504647e-15 0.015799999999995956168 -0.065000000000000793254 rpy=-1.5707963267948983344 -0.78539816339744794593 -8.4801163929695123491e-15 -> xyz=-1.3322676295501878485e-15 0.015799999999994734923 -0.065000000000000376921 rpy=-1.57079632679489678 -0.78539816339744150664 -8.5144621655032178393e-15
- joint LL_HR: origin xyz=-1.5249813257468713577e-16 0.069999999999999895639 -4.8559453586656778667e-17 rpy=-5.5967126325698482102e-15 0.78539816339745760487 -7.914946909686092054e-15 -> xyz=-1.5163483659484564161e-16 0.069999999999999895639 -4.8559453586656402725e-17 rpy=1.3339637907287298868e-27 0.78539816339744794593 1.2332799712965867172e-17
- joint LL_KFE: origin xyz=-0.22000000000000025091 9.5826124812958823895e-15 0.074199999999999988187 rpy=1.004141528052162953e-27 -1.9324819522386478582e-15 0 -> xyz=-0.2200000000000001954 9.5826124812958823895e-15 0.074199999999999946554 rpy=2.3904489498968254871e-15 1.85268467234245216e-15 -1.2267964422107583764e-14
- joint LR_FAA: origin xyz=-1.1102230246251565404e-16 0.020000000000011272649 -1.1102230246251565404e-15 rpy=-1.570796326794896558 -1.5707963267948952257 0 -> xyz=0 0.020000000000011272649 -1.1379786002407854539e-15 rpy=-1.5707963267948958919 -1.570796326794896336 0
- joint LR_FFE: origin xyz=-0.17999999999999954925 -2.6888213877640509963e-16 1.3877787807814456755e-16 rpy=1.3641350715342211265e-16 -1.3045120539345628793e-15 -1.1124684032044933672e-16 -> xyz=-0.18000000000000010436 -3.2265856653168611956e-16 1.3877787807814456755e-16 rpy=4.6473388338391139794e-16 1.3322676295501568857e-15 -1.0785973072212841079e-15
- joint LR_FOOT_frame: origin xyz=-7.771561172376095783e-16 -0.032999999999999585221 0.020976404179758215834 rpy=-1.570796326794896558 -1.570796326794896558 0 -> xyz=-7.4940054162198066479e-16 -0.032999999999999585221 0.020976404179758215834 rpy=-1.570796326794896558 -1.570796326794896558 0
- joint LR_HAA: origin xyz=0.015799999999996518218 -3.8857805861880478915e-16 -0.064999999999998905875 rpy=-2.9423517219288057983e-15 -1.5707963267948932273 0 -> xyz=0.015799999999996230254 1.3461454173580023053e-15 -0.064999999999997726263 rpy=-2.5294501794417421484e-15 -1.5707963267948930053 0
- joint LR_HFE: origin xyz=-5.7037707890117417264e-15 -0.015799999999999800315 -0.064999999999993979261 rpy=-1.5707963267948923392 -0.78539816339744894513 -6.4495050167007133749e-15 -> xyz=-6.5503158452884235885e-15 -0.015800000000000355427 -0.064999999999994145794 rpy=-1.570796326794891673 -0.78539816339743961926 -6.3317480822993795962e-15
- joint LR_HR: origin xyz=-1.7663949738338549142e-16 -0.070000000000000103806 -5.9783511249299864752e-17 rpy=4.5998802503059629481e-17 0.78539816339744816798 6.5052130350937854523e-17 -> xyz=-1.7663949738338549142e-16 -0.070000000000000103806 -5.9783511249299827774e-17 rpy=-4.767057147862150383e-16 0.78539816339744816798 -6.741636871132349286e-16
- joint LR_KFE: origin xyz=-0.21999999999999950151 5.2510079617817950748e-15 -0.074199999999999738387 rpy=-8.3136953572731735262e-16 -1.537353622424777934e-15 -1.6653345369376596223e-16 -> xyz=-0.22000000000000236033 5.4522358849951046977e-15 -0.074200000000000695954 rpy=-6.6483608203348963737e-16 -1.5373536224247637345e-15 -8.6042284408420128485e-16

Commit message: Add Gazebo tags

File: urdf/robot.urdf (robot description, URDF)
Before this commit: robot onshape, 15 links, 14 joints
Links:
- link ll_faa: mass 0.19869955000000011358 -> 0.19869954999999991929
- link ll_ffe: mass 0.099322750000000056825 -> 0.099322750000000042947
- link ll_haa: mass 0.79600000000000059597 -> 0.7960000000000012621
- link ll_hfe: mass 3.5233394799999966374 -> 3.5233394799999935287
- link ll_hr: mass 0.73133287000000013478 -> 0.73133287000000068989
- link ll_kfe: mass 0.24071601000000006354 -> 0.24071601000000050763
- link lr_faa: mass 0.19869955000000000256 -> 0.1986995499999999748
- link lr_haa: mass 0.79599999999999970779 -> 0.79599999999999948574
- link lr_hfe: mass 2.4960000000000079901 -> 2.4960000000000071019
- link lr_hr: mass 0.73133287000000080091 -> 0.73133287000000057887
- link lr_kfe: mass 0.24099999999999996425 -> 0.24100000000000004752
- link torso: mass 2.927037159999976268 -> 2.9270371599999869261; geometry collision box size=0.17999999999999999334 0.25 0.25; visual mesh filename=package://cal_hum_description/meshs/torso.stl
Joints:
- joint LL_FAA: origin xyz=6.6613381477509392425e-16 0.020000000000026579849 -1.9428902930940239457e-15 rpy=-1.5707963267948634734 -1.5707963267948870101 0 -> xyz=-2.2204460492503130808e-16 0.020000000000026614544 -2.8588242884097780916e-15 rpy=-1.570796326794896558 -1.5707963267948870101 0
- joint LL_FFE: origin xyz=-0.18000000000000204725 7.6709472107694409715e-15 -4.5519144009631418157e-15 rpy=-4.142519660632226433e-15 -2.2343238370579094176e-15 5.9396931817444589069e-15 -> xyz=-0.18000000000000104805 7.6379874647258816367e-15 -3.5527136788005009294e-15 rpy=-4.7237149809748546698e-16 1.4636729328685165243e-17 -2.1608234000908133641e-17
- joint LL_FOOT_frame: origin xyz=1.360023205165816762e-15 -0.033000000000000473399 0.020976404179762330598 rpy=-1.5707963267948936714 -1.570796326794896558 0 -> xyz=1.360023205165816762e-15 -0.033000000000000473399 0.020976404179762337537 rpy=-1.570796326794896558 -1.570796326794896558 0
- joint LL_HAA: origin xyz=0.015799999999996153927 -1.360023205165816762e-15 -0.064999999999997906674 rpy=1.2864546617328002073e-15 -1.5707963267948952257 0 -> xyz=0.01579999999999582086 -1.8596235662471372052e-15 -0.06499999999999730993 rpy=9.9396442047859508385e-16 -1.5707963267948770181 0
- joint LL_HFE: origin xyz=-1.3322676295501878485e-15 0.015799999999994734923 -0.065000000000000376921 rpy=-1.57079632679489678 -0.78539816339744150664 -8.5144621655032178393e-15 -> xyz=-1.7902346272080649214e-15 0.015799999999995956168 -0.065000000000000807132 rpy=-1.57079632679489678 -0.78539816339745571749 -2.5516191694803642929e-14
- joint LL_HR: origin xyz=-1.5163483659484564161e-16 0.069999999999999895639 -4.8559453586656402725e-17 rpy=1.3339637907287298868e-27 0.78539816339744794593 1.2332799712965867172e-17 -> xyz=-1.5249813257468723438e-16 0.069999999999999895639 -4.8559453586656408888e-17 rpy=-1.1530883081439468873e-16 0.78539816339745505136 -3.9899370513288793298e-16
- joint LL_KFE: origin xyz=-0.2200000000000001954 9.5826124812958823895e-15 0.074199999999999946554 rpy=2.3904489498968254871e-15 1.85268467234245216e-15 -1.2267964422107583764e-14 -> xyz=-0.21999999999999791944 1.0247011572594999507e-14 0.074199999999998045297 rpy=9.0122625749589332474e-16 -9.6855554553076782161e-15 -1.1275702593848007602e-15
- joint LR_FAA: origin xyz=0 0.020000000000011272649 -1.1379786002407854539e-15 rpy=-1.5707963267948958919 -1.570796326794896336 0 -> xyz=0 0.020000000000011439183 -1.1379786002407854539e-15 rpy=-1.5707963267948961139 -1.5707963267948961139 0
- joint LR_FFE: origin xyz=-0.18000000000000010436 -3.2265856653168611956e-16 1.3877787807814456755e-16 rpy=4.6473388338391139794e-16 1.3322676295501568857e-15 -1.0785973072212841079e-15 -> xyz=-0.18000000000000010436 -3.2265856653168611956e-16 1.1102230246251565404e-16 rpy=4.9088374165698854435e-16 9.020562075078750025e-16 4.9379514839931034925e-16
- joint LR_FOOT_frame: origin xyz=-7.4940054162198066479e-16 -0.032999999999999585221 0.020976404179758215834 rpy=-1.570796326794896558 -1.570796326794896558 0 -> xyz=-6.9388939039072283776e-16 -0.032999999999999141131 0.020976404179758219304 rpy=-1.570796326794896558 -1.570796326794896558 0
- joint LR_HFE: origin xyz=-6.5503158452884235885e-15 -0.015800000000000355427 -0.064999999999994145794 rpy=-1.570796326794891673 -0.78539816339743961926 -6.3317480822993795962e-15 -> xyz=-6.8417493892525271804e-15 -0.015800000000001562794 -0.064999999999994256816 rpy=-1.570796326794891673 -0.78539816339744905616 -6.3317480822994348165e-15
- joint LR_KFE: origin xyz=-0.22000000000000236033 5.4522358849951046977e-15 -0.074200000000000695954 rpy=-6.6483608203348963737e-16 -1.5373536224247637345e-15 -8.6042284408420128485e-16 -> xyz=-0.21999999999999936273 5.1399856593192794207e-15 -0.074199999999999738387 rpy=-6.6483608203348431256e-16 -1.5373536224247538737e-15 8.165942964201880017e-31

Commit message: First successfully running in Gazebo

File: urdf/robot.urdf (robot description, URDF)
Before this commit: robot onshape, 15 links, 14 joints
Joints:
- joint LL_FFE: limit lower=-0.52359877559829881566 upper=1.2217304763960306069 effort=60 velocity=20 -> lower=-1.52359877559829881566 upper=1.2217304763960306069 effort=60 velocity=20
- joint LL_KFE: limit lower=0 upper=2.0943951023931952626 effort=120 velocity=14 -> lower=0.1 upper=2.0943951023931952626 effort=120 velocity=14
- joint LR_FFE: limit lower=-0.52359877559829881566 upper=1.2217304763960306069 effort=60 velocity=23 -> lower=-1.52359877559829881566 upper=1.2217304763960306069 effort=60 velocity=23
- joint LR_KFE: limit lower=0 upper=2.0943951023931952626 effort=120 velocity=14 -> lower=0.1 upper=2.0943951023931952626 effort=120 velocity=14

Commit message: Add more collision shapes

File: urdf/robot.urdf (robot description, URDF)
Before this commit: robot onshape, 15 links, 14 joints
Links:
- link ll_hfe: geometry collision cylinder length=0.080000000000000001665 radius=0.051999999999999997613; collision cylinder length=0.089999999999999996669 radius=0.061499999999999999112
- link ll_kfe: geometry collision box size=0.02999999999999999889 0.040000000000000000833 0.1600000000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; visual mesh filename=package://cal_hum_description/meshs/ll_kfe.stl
- link lr_hfe: geometry collision cylinder length=0.080000000000000001665 radius=0.051999999999999997613; collision cylinder length=0.089999999999999996669 radius=0.061499999999999999112
- link lr_kfe: geometry collision box size=0.02999999999999999889 0.040000000000000000833 0.1600000000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; visual mesh filename=package://cal_hum_description/meshs/lr_kfe.stl
Joints:
- joint LL_KFE: limit lower=0.1 upper=2.0943951023931952626 effort=120 velocity=14 -> lower=0 upper=2.0943951023931952626 effort=120 velocity=14
- joint LR_KFE: limit lower=0.1 upper=2.0943951023931952626 effort=120 velocity=14 -> lower=0 upper=2.0943951023931952626 effort=120 velocity=14

Commit message: Update urdf

File: urdf/robot.urdf (robot description, URDF)
Before this commit: robot onshape, 15 links, 14 joints
Links:
- link ll_faa: mass 0.19869954999999991929 -> 0.46714990999999994603; geometry collision box size=0.16000000000000000333 0.055000000000000000278 0.0550000000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; visual mesh filename=package://cal_hum_description/meshs/ll_faa.stl
- link ll_ffe: mass 0.099322750000000042947 -> 0.099322750000000015191
- link ll_haa: mass 0.7960000000000012621 -> 0.85100000000001196909
- link ll_hfe: mass 3.5233394799999935287 -> 2.2535340099999987551
- link ll_hr: mass 0.73133287000000068989 -> 0.75099999999998401368
- link ll_kfe: mass 0.24071601000000050763 -> 0.24071601000000042436
- link lr_faa: mass 0.1986995499999999748 -> 0.46714991000000016808; geometry collision box size=0.16000000000000000333 0.055000000000000000278 0.0550000000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; visual mesh filename=package://cal_hum_description/meshs/lr_faa.stl
- link lr_ffe: mass 0.099322280000000012778 -> 0.099322280000000026656
- link lr_haa: mass 0.79599999999999948574 -> 0.79600000000000414868
- link lr_hfe: mass 2.4960000000000071019 -> 2.2540000000000013358
- link lr_hr: mass 0.73133287000000057887 -> 0.75099999999998801048
- link lr_kfe: mass 0.24100000000000004752 -> 0.24099999999999988098
- link torso: mass 2.9270371599999869261 -> 5.3781180999999937953
Joints:
- joint LL_FAA: origin xyz=-2.2204460492503130808e-16 0.020000000000026614544 -2.8588242884097780916e-15 rpy=-1.570796326794896558 -1.5707963267948870101 0 -> xyz=8.8817841970012523234e-16 0.019999999999998921418 1.0269562977782697999e-15 rpy=-1.5707963267947515629 -1.4450247660621533541 -1.1629114424755023013e-13
- joint LL_FFE: limit lower=-1.52359877559829881566 upper=1.2217304763960306069 effort=60 velocity=20 -> lower=-0.52359877559829881566 upper=1.2217304763960306069 effort=60 velocity=20; origin xyz=-0.18000000000000104805 7.6379874647258816367e-15 -3.5527136788005009294e-15 rpy=-4.7237149809748546698e-16 1.4636729328685165243e-17 -2.1608234000908133641e-17 -> xyz=-0.18000000000000204725 4.0648040489088543836e-13 -4.4131365228849972482e-15 rpy=-4.9741081456802783629e-15 -7.8078125061771119145e-15 -0.3496172140838589848
- joint LL_FOOT_frame: origin xyz=1.360023205165816762e-15 -0.033000000000000473399 0.020976404179762337537 rpy=-1.570796326794896558 -1.570796326794896558 0 -> xyz=5.0760714645492477359e-08 -0.048285133326044726854 0.01182062398699337824 rpy=3.1415926535897913396 -1.3962634015954631383 1.570796326794896558
- joint LL_HAA: origin xyz=0.01579999999999582086 -1.8596235662471372052e-15 -0.06499999999999730993 rpy=9.9396442047859508385e-16 -1.5707963267948770181 0 -> xyz=0.015799999999996344746 -3.7470027081099033239e-16 -0.064999999999999613642 rpy=-1.5707963267949045516 -1.4678600129856298473 1.570796326794289488
- joint LL_HFE: origin xyz=-1.7902346272080649214e-15 0.015799999999995956168 -0.065000000000000807132 rpy=-1.57079632679489678 -0.78539816339745571749 -2.5516191694803642929e-14 -> xyz=1.1102230246251565404e-16 0.015799999999995040234 -0.064999999999999308331 rpy=-1.5707963267948641395 -1.2485808691306654605 -4.5486223788766130327e-14
- joint LL_HR: origin xyz=-1.5249813257468723438e-16 0.069999999999999895639 -4.8559453586656408888e-17 rpy=-1.1530883081439468873e-16 0.78539816339745505136 -3.9899370513288793298e-16 -> xyz=-1.6696713456276768284e-16 0.069999999999999909517 -4.8572257327350598644e-17 rpy=-0.072206686120917601412 0.78278216060187066905 -0.10220480535128237398
- joint LL_KFE: origin xyz=-0.21999999999999791944 1.0247011572594999507e-14 0.074199999999998045297 rpy=9.0122625749589332474e-16 -9.6855554553076782161e-15 -1.1275702593848007602e-15 -> xyz=-0.2200000000000001954 5.0049547839492447565e-13 0.074199999999999807776 rpy=-1.1996374222978450601e-14 3.4286500686111271094e-14 0.98360185480604667152
- joint LR_FAA: origin xyz=0 0.020000000000011439183 -1.1379786002407854539e-15 rpy=-1.5707963267948961139 -1.5707963267948961139 0 -> xyz=1.6653345369377348106e-16 0.020000000000000323075 -1.9428902930940239457e-16 rpy=1.5707963267948852337 -1.4450247661876081118 -3.1415926535897811256
- joint LR_FFE: limit lower=-1.52359877559829881566 upper=1.2217304763960306069 effort=60 velocity=23 -> lower=-0.52359877559829881566 upper=1.2217304763960306069 effort=60 velocity=23; origin xyz=-0.18000000000000010436 -3.2265856653168611956e-16 1.1102230246251565404e-16 rpy=4.9088374165698854435e-16 9.020562075078750025e-16 4.9379514839931034925e-16 -> xyz=-0.18000000000000068723 -1.6653345369377348106e-16 8.3266726846886740532e-17 rpy=1.1209570441384864999e-15 1.4760710728832299551e-15 -0.34961721405632484316
- joint LR_FOOT_frame: origin xyz=-6.9388939039072283776e-16 -0.032999999999999141131 0.020976404179758219304 rpy=-1.570796326794896558 -1.570796326794896558 0 -> xyz=5.0760711800545976757e-08 -0.048285133326043450097 0.011820623986989048371 rpy=-3.141592653589793116 -1.3962634015954631383 1.570796326794896558
- joint LR_HAA: origin xyz=0.015799999999996230254 1.3461454173580023053e-15 -0.064999999999997726263 rpy=-2.5294501794417421484e-15 -1.5707963267948930053 0 -> xyz=0.015799999999996486993 -2.7755575615628913511e-16 -0.064999999999999238942 rpy=1.5707963267948976682 -1.4678600130881280794 -1.5707963267948414909
- joint LR_HFE: origin xyz=-6.8417493892525271804e-15 -0.015800000000001562794 -0.064999999999994256816 rpy=-1.570796326794891673 -0.78539816339744905616 -6.3317480822994348165e-15 -> xyz=-1.2836953722228372499e-15 -0.015800000000000161138 -0.064999999999999391598 rpy=-1.5707963267948925612 -1.2485808690947428623 -6.3154349151414743693e-15
- joint LR_HR: origin xyz=-1.7663949738338549142e-16 -0.070000000000000103806 -5.9783511249299827774e-17 rpy=-4.767057147862150383e-16 0.78539816339744816798 -6.741636871132349286e-16 -> xyz=-1.9472271017839659635e-16 -0.070000000000000103806 -5.290906601729261638e-17 rpy=0.07220668604874565244 0.78278216060711247604 0.10220480524894931529
- joint LR_KFE: origin xyz=-0.21999999999999936273 5.1399856593192794207e-15 -0.074199999999999738387 rpy=-6.6483608203348431256e-16 -1.5373536224247538737e-15 8.165942964201880017e-31 -> xyz=-0.21999999999999936273 7.403799795469012679e-15 -0.074199999999999266542 rpy=-2.4715536250851352852e-15 3.1294003481309170141e-15 0.9836018547500596787
