Commit message: Update urdf

File: urdf/robot.urdf (robot description, URDF)
Before this commit: robot onshape, 15 links, 14 joints
Links:
- link ll_faa: mass 0.46714990999999994603 -> 0.46714990999999950194
- link ll_ffe: mass 0.099322750000000015191 -> 0.099322750000000056825
- link ll_haa: mass 0.85100000000001196909 -> 0.85100000000001085887
- link ll_hfe: mass 2.2535340099999987551 -> 2.2535340100000000874
- link ll_hr: mass 0.75099999999998401368 -> 0.75099999999998279243
- link ll_kfe: mass 0.24071601000000042436 -> 0.24071601000000064641
- link lr_faa: mass 0.46714991000000016808 -> 0.46714990999999983501
- link lr_haa: mass 0.79600000000000414868 -> 0.79600000000000059597
- link lr_hfe: mass 2.2540000000000013358 -> 2.2540000000000004476
- link lr_hr: mass 0.75099999999998801048 -> 0.75099999999999023093
- link lr_kfe: mass 0.24099999999999988098 -> 0.24100000000000007527
- link torso: mass 5.3781180999999937953 -> 5.3781180999999893544
Joints:
- joint LL_FAA: origin xyz=8.8817841970012523234e-16 0.019999999999998921418 1.0269562977782697999e-15 rpy=-1.5707963267947515629 -1.4450247660621533541 -1.1629114424755023013e-13 -> xyz=7.771561172376095783e-16 0.019999999999998924888 1.0824674490095276269e-15 rpy=-1.5707963267948970021 -1.570796326794876574 0
- joint LL_FFE: origin xyz=-0.18000000000000204725 4.0648040489088543836e-13 -4.4131365228849972482e-15 rpy=-4.9741081456802783629e-15 -7.8078125061771119145e-15 -0.3496172140838589848 -> xyz=-0.18000000000000221378 4.0657234523511220914e-13 -4.3853809472693683347e-15 rpy=4.1335758622659789005e-30 1.5777218104420236108e-30 -6.383782391594657996e-15
- joint LL_FOOT_frame: origin xyz=5.0760714645492477359e-08 -0.048285133326044726854 0.01182062398699337824 rpy=3.1415926535897913396 -1.3962634015954631383 1.570796326794896558 -> xyz=5.0760714742636992014e-08 -0.048285133326044671342 0.011820623986993364363 rpy=3.1415926535897846783 -1.3962634015954633604 1.570796326794896558
- joint LL_HAA: origin xyz=0.015799999999996344746 -3.7470027081099033239e-16 -0.064999999999999613642 rpy=-1.5707963267949045516 -1.4678600129856298473 1.570796326794289488 -> xyz=0.015799999999996330868 -3.1918911957973250537e-16 -0.064999999999999613642 rpy=-2.9816562105458668087e-15 -1.5707963267948934494 0
- joint LL_HFE: origin xyz=1.1102230246251565404e-16 0.015799999999995040234 -0.064999999999999308331 rpy=-1.5707963267948641395 -1.2485808691306654605 -4.5486223788766130327e-14 -> xyz=-8.3266726846886740532e-17 0.015799999999994970845 -0.064999999999999710787 rpy=-1.5707963267948823471 -0.78539816339744961127 3.2543908859931252475e-15
- joint LL_HR: origin xyz=-1.6696713456276768284e-16 0.069999999999999909517 -4.8572257327350598644e-17 rpy=-0.072206686120917601412 0.78278216060187066905 -0.10220480535128237398 -> xyz=-1.6653345369377348106e-16 0.069999999999999854006 -4.8572257327350598644e-17 rpy=6.776315175848504861e-28 0.78539816339744950024 4.7915784122997950057e-28
- joint LL_KFE: origin xyz=-0.2200000000000001954 5.0049547839492447565e-13 0.074199999999999807776 rpy=-1.1996374222978450601e-14 3.4286500686111271094e-14 0.98360185480604667152 -> xyz=-0.22000000000000022315 5.0043823252021724102e-13 0.074199999999999863287 rpy=-3.3760985920712169733e-14 7.3374569801132745765e-15 6.4670491184412426029e-15
- joint LR_FAA: origin xyz=1.6653345369377348106e-16 0.020000000000000323075 -1.9428902930940239457e-16 rpy=1.5707963267948852337 -1.4450247661876081118 -3.1415926535897811256 -> xyz=-4.5519144009631418157e-15 0.020000000000000892064 -3.1641356201816961402e-15 rpy=-1.570796326794896558 -1.5707963267948958919 0
- joint LR_FFE: origin xyz=-0.18000000000000068723 -1.6653345369377348106e-16 8.3266726846886740532e-17 rpy=1.1209570441384864999e-15 1.4760710728832299551e-15 -0.34961721405632484316 -> xyz=-0.18000000000000015987 -3.2439329000766292666e-16 1.6653345369377348106e-16 rpy=2.8414770536498554039e-15 2.1649348980189791287e-15 1.9428902930938756399e-15
- joint LR_FOOT_frame: origin xyz=5.0760711800545976757e-08 -0.048285133326043450097 0.011820623986989048371 rpy=-3.141592653589793116 -1.3962634015954631383 1.570796326794896558 -> xyz=5.0760711967079430451e-08 -0.048285133326045004409 0.011820623986989381438 rpy=3.141592653589793116 -1.3962634015954633604 1.570796326794896558
- joint LR_HAA: origin xyz=0.015799999999996486993 -2.7755575615628913511e-16 -0.064999999999999238942 rpy=1.5707963267948976682 -1.4678600130881280794 -1.5707963267948414909 -> xyz=0.01579999999999619556 1.193489751472043281e-15 -0.064999999999998087086 rpy=-1.6145151215107273488e-15 -1.5707963267948941155 0
- joint LR_HFE: origin xyz=-1.2836953722228372499e-15 -0.015800000000000161138 -0.064999999999999391598 rpy=-1.5707963267948925612 -1.2485808690947428623 -6.3154349151414743693e-15 -> xyz=-1.8873791418627661187e-15 -0.015799999999999994604 -0.064999999999998808731 rpy=-1.5707963267948912289 -0.78539816339743961926 -3.2139718585574148952e-15
- joint LR_HR: origin xyz=-1.9472271017839659635e-16 -0.070000000000000103806 -5.290906601729261638e-17 rpy=0.07220668604874565244 0.78278216060711247604 0.10220480524894931529 -> xyz=-1.9428902930940239457e-16 -0.070000000000000062172 -5.5511151231257808532e-17 rpy=-6.2032260096825242622e-16 0.7853981633974492782 -8.7726863533765840477e-16
- joint LR_KFE: origin xyz=-0.21999999999999936273 7.403799795469012679e-15 -0.074199999999999266542 rpy=-2.4715536250851352852e-15 3.1294003481309170141e-15 0.9836018547500596787 -> xyz=-0.21999999999999927947 7.3118594512422419029e-15 -0.074199999999999377565 rpy=-5.5888040731323801616e-15 -1.6961427793646633868e-16 -4.357625371653309492e-15

Commit message: Update the defaultJointState

File: urdf/robot.urdf (robot description, URDF)
Before this commit: robot onshape, 15 links, 14 joints
Joints:
- joint LL_KFE: limit lower=0 upper=2.0943951023931952626 effort=120 velocity=14 -> lower=0.1 upper=2.0943951023931952626 effort=120 velocity=14
- joint LR_KFE: limit lower=0 upper=2.0943951023931952626 effort=120 velocity=14 -> lower=0.1 upper=2.0943951023931952626 effort=120 velocity=14

Commit message: New ankle, small torque

File: urdf/robot.urdf (robot description, URDF)
Before this commit: robot onshape, 15 links, 14 joints
Links:
- link ll_faa: mass 0.46714990999999950194 -> 0.50700000000000067235; geometry collision box size=0.16000000000000000333 0.055000000000000000278 0.0120000000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; collision cylinder length=0.06500000000000000222 radius=0.026999999999999999695
- link ll_haa: mass 0.85100000000001085887 -> 0.89699999999999757705; geometry collision cylinder length=0.050000000000000002776 radius=0.055000000000000000278; visual mesh filename=package://cal_hum_description/meshs/ll_haa.stl
- link ll_hfe: mass 2.2535340100000000874 -> 2.6890000000000013891
- link ll_hr: mass 0.75099999999998279243 -> 0.7970000000000008189
- link ll_kfe: mass 0.24071601000000064641 -> 0.3499999999999999778
- link lr_faa: mass 0.46714990999999983501 -> 0.50700000000000011724; geometry collision box size=0.16000000000000000333 0.055000000000000000278 0.0120000000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; collision cylinder length=0.06500000000000000222 radius=0.026999999999999999695
- link lr_ffe: mass 0.099322280000000026656 -> 0.099322280000000040534
- link lr_haa: mass 0.79600000000000059597 -> 0.89700000000000745803; geometry collision cylinder length=0.050000000000000002776 radius=0.055000000000000000278; visual mesh filename=package://cal_hum_description/meshs/lr_haa.stl
- link lr_hfe: mass 2.2540000000000004476 -> 2.6890000000000005009
- link lr_hr: mass 0.75099999999999023093 -> 0.79699999999999693312
- link lr_kfe: mass 0.24100000000000007527 -> 0.3499999999999999778
- link torso: mass 5.3781180999999893544 -> 5.378118099999987578
Joints:
- joint LL_FAA: limit lower=-0.52359877559829881566 upper=0.52359877559829881566 effort=18 velocity=42 -> lower=-0.52359877559829881566 upper=0.52359877559829881566 effort=5 velocity=42; origin xyz=7.771561172376095783e-16 0.019999999999998924888 1.0824674490095276269e-15 rpy=-1.5707963267948970021 -1.570796326794876574 0 -> xyz=-3.6637359812630165834e-15 0.017499999999998770012 -3.8857805861880478915e-16 rpy=-1.5707963267948938935 -1.5707963267948830133 0
- joint LL_FFE: limit lower=-0.52359877559829881566 upper=1.2217304763960306069 effort=60 velocity=20 -> lower=-0.52359877559829881566 upper=0.69813170079773179122 effort=20 velocity=20; origin xyz=-0.18000000000000221378 4.0657234523511220914e-13 -4.3853809472693683347e-15 rpy=4.1335758622659789005e-30 1.5777218104420236108e-30 -6.383782391594657996e-15 -> xyz=-0.18000000000000221378 4.0657234523511220914e-13 -4.4131365228849972482e-15 rpy=1.1476240689710679376e-27 8.5046658791676055396e-29 8.3266726846923028133e-17
- joint LL_FOOT_frame: origin xyz=5.0760714742636992014e-08 -0.048285133326044671342 0.011820623986993364363 rpy=3.1415926535897846783 -1.3962634015954633604 1.570796326794896558 -> xyz=5.8564264548977007507e-15 -0.048688979881312266507 0.014485028526583749314 rpy=3.141592653589793116 -1.3962634015954653588 1.570796326794896558
- joint LL_HAA: limit lower=-0.52359877559829881566 upper=0.785398163397448279 effort=60 velocity=23 -> lower=-0.61086523819801530344 upper=0.61086523819801530344 effort=20 velocity=23; origin xyz=0.015799999999996330868 -3.1918911957973250537e-16 -0.064999999999999613642 rpy=-2.9816562105458668087e-15 -1.5707963267948934494 0 -> xyz=0.015799999999996268418 -2.7755575615628913511e-16 -0.064999999999999849565 rpy=-3.9874966918901588628e-15 -1.5707963267948950037 0
- joint LL_HFE: limit lower=-1.9198621771937625091 upper=1.9198621771937625091 effort=90 velocity=20 -> lower=-1.7453292519943295336 upper=0.52359877559829881566 effort=30 velocity=20; origin xyz=-8.3266726846886740532e-17 0.015799999999994970845 -0.064999999999999710787 rpy=-1.5707963267948823471 -0.78539816339744961127 3.2543908859931252475e-15 -> xyz=2.6367796834847467835e-16 0.015799999999994956967 -0.064999999999999530376 rpy=-1.5707963267948812369 -0.78539816339744850104 7.0425066851191171402e-15
- joint LL_HR: limit lower=-0.52359877559829881566 upper=1.0471975511965976313 effort=60 velocity=23 -> lower=-0.61086523819801530344 upper=0.61086523819801530344 effort=20 velocity=23; origin xyz=-1.6653345369377348106e-16 0.069999999999999854006 -4.8572257327350598644e-17 rpy=6.776315175848504861e-28 0.78539816339744950024 4.7915784122997950057e-28 -> xyz=-1.6653345369377348106e-16 0.069999999999999854006 -4.8572257327350610969e-17 rpy=4.2686888720530165754e-16 0.78539816339746193474 2.380040609040672766e-15
- joint LL_KFE: limit lower=0.1 upper=2.0943951023931952626 effort=120 velocity=14 -> lower=0 upper=2.0943951023931952626 effort=30 velocity=14; origin xyz=-0.22000000000000022315 5.0043823252021724102e-13 0.074199999999999863287 rpy=-3.3760985920712169733e-14 7.3374569801132745765e-15 6.4670491184412426029e-15 -> xyz=-0.21999999999999989009 5.0031506715342288771e-13 0.074199999999999918798 rpy=-3.6817022053377870126e-14 8.7267374499327085356e-15 1.9428902930912523323e-16
- joint LR_FAA: limit lower=-0.52359877559829881566 upper=0.52359877559829881566 effort=18 velocity=42 -> lower=-0.52359877559829881566 upper=0.52359877559829881566 effort=5 velocity=42; origin xyz=-4.5519144009631418157e-15 0.020000000000000892064 -3.1641356201816961402e-15 rpy=-1.570796326794896558 -1.5707963267948958919 0 -> xyz=7.771561172376095783e-16 0.017500000000000015543 -9.1593399531575414585e-16 rpy=-1.570796326794896336 -1.5707963267948850117 0
- joint LR_FFE: limit lower=-0.52359877559829881566 upper=1.2217304763960306069 effort=60 velocity=23 -> lower=-0.52359877559829881566 upper=0.69813170079773179122 effort=20 velocity=23; origin xyz=-0.18000000000000015987 -3.2439329000766292666e-16 1.6653345369377348106e-16 rpy=2.8414770536498554039e-15 2.1649348980189791287e-15 1.9428902930938756399e-15 -> xyz=-0.1800000000000017697 2.9490299091605720605e-17 -9.7144514654701197287e-16 rpy=-2.4605607242230561785e-15 -2.1937466413332281916e-15 -2.4980018054056664297e-16
- joint LR_FOOT_frame: origin xyz=5.0760711967079430451e-08 -0.048285133326045004409 0.011820623986989381438 rpy=3.141592653589793116 -1.3962634015954633604 1.570796326794896558 -> xyz=-2.7755575615628913511e-16 -0.048688979881310823217 0.014485028526582469088 rpy=-3.141592653589793116 -1.3962634015954653588 1.570796326794896558
- joint LR_HAA: limit lower=-1.0471975511965976313 upper=0.52359877559829881566 effort=60 velocity=23 -> lower=-0.61086523819801530344 upper=0.61086523819801530344 effort=20 velocity=23; origin xyz=0.01579999999999619556 1.193489751472043281e-15 -0.064999999999998087086 rpy=-1.6145151215107273488e-15 -1.5707963267948941155 0 -> xyz=0.015799999999996469646 -2.9143354396410359186e-16 -0.064999999999999238942 rpy=-2.3800406090414426943e-15 -1.5707963267948694686 0
- joint LR_HFE: limit lower=-1.9198621771937625091 upper=1.9198621771937625091 effort=90 velocity=20 -> lower=-1.7453292519943295336 upper=0.52359877559829881566 effort=30 velocity=20; origin xyz=-1.8873791418627661187e-15 -0.015799999999999994604 -0.064999999999998808731 rpy=-1.5707963267948912289 -0.78539816339743961926 -3.2139718585574148952e-15 -> xyz=-1.0130785099704553431e-15 -0.015799999999999869704 -0.064999999999998711586 rpy=-1.570796326794891673 -0.78539816339745049945 2.2818401626814027346e-14
- joint LR_HR: limit lower=-1.0471975511965976313 upper=0.52359877559829881566 effort=60 velocity=23 -> lower=-0.61086523819801530344 upper=0.61086523819801530344 effort=20 velocity=23; origin xyz=-1.9428902930940239457e-16 -0.070000000000000062172 -5.5511151231257808532e-17 rpy=-6.2032260096825242622e-16 0.7853981633974492782 -8.7726863533765840477e-16 -> xyz=1.1232681451645076202e-15 -0.070000000000000575651 1.4718781748967987512e-15 rpy=1.4130832128180086564e-15 0.7853981633974472798 -8.3266726844983662902e-17
- joint LR_KFE: limit lower=0.1 upper=2.0943951023931952626 effort=120 velocity=14 -> lower=0 upper=2.0943951023931952626 effort=30 velocity=14; origin xyz=-0.21999999999999927947 7.3118594512422419029e-15 -0.074199999999999377565 rpy=-5.5888040731323801616e-15 -1.6961427793646633868e-16 -4.357625371653309492e-15 -> xyz=-0.21999999999999853006 7.7264583620006987985e-15 -0.074199999999998419997 rpy=1.2766813666707529471e-14 1.7506442815481622092e-15 -4.7184478546574556665e-16

Commit message: Rename verything to berkeley_humanoid

File: urdf/robot.urdf (robot description, URDF)
Before this commit: robot onshape, 15 links, 14 joints
Links:
- link ll_faa: geometry collision box size=0.16000000000000000333 0.055000000000000000278 0.0120000000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; collision cylinder length=0.06500000000000000222 radius=0.026999999999999999695
- link ll_ffe: geometry visual mesh filename=package://berkeley_humanoid_description/meshs/ll_ffe.stl
- link ll_haa: geometry collision cylinder length=0.050000000000000002776 radius=0.055000000000000000278; visual mesh filename=package://berkeley_humanoid_description/meshs/ll_haa.stl
- link ll_hfe: geometry collision cylinder length=0.080000000000000001665 radius=0.051999999999999997613; collision cylinder length=0.089999999999999996669 radius=0.061499999999999999112
- link ll_hr: geometry visual mesh filename=package://berkeley_humanoid_description/meshs/ll_hr.stl
- link ll_kfe: geometry collision box size=0.02999999999999999889 0.040000000000000000833 0.1600000000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; visual mesh filename=package://berkeley_humanoid_description/meshs/ll_kfe.stl
- link lr_faa: geometry collision box size=0.16000000000000000333 0.055000000000000000278 0.0120000000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; collision cylinder length=0.06500000000000000222 radius=0.026999999999999999695
- link lr_ffe: geometry visual mesh filename=package://berkeley_humanoid_description/meshs/lr_ffe.stl
- link lr_haa: geometry collision cylinder length=0.050000000000000002776 radius=0.055000000000000000278; visual mesh filename=package://berkeley_humanoid_description/meshs/lr_haa.stl
- link lr_hfe: geometry collision cylinder length=0.080000000000000001665 radius=0.051999999999999997613; collision cylinder length=0.089999999999999996669 radius=0.061499999999999999112
- link lr_hr: geometry visual mesh filename=package://berkeley_humanoid_description/meshs/lr_hr.stl
- link lr_kfe: geometry collision box size=0.02999999999999999889 0.040000000000000000833 0.1600000000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; visual mesh filename=package://berkeley_humanoid_description/meshs/lr_kfe.stl
- link torso: geometry collision box size=0.17999999999999999334 0.25 0.25; visual mesh filename=package://berkeley_humanoid_description/meshs/torso.stl
